File: GSMshield.sch (EAGLE design)
At the start: 65 parts, among them IC1 RT8289, IC2 SIM900, J1 SIM Socket, J2 Antenna, J3 Breakout 1, J4 Breakout 2, J5 ARDUINO-SHIELD_R3, Q1 2N7002, Q2 2N7002, Q3 2N7002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

Commit message: Changed all fonts to vector Increased VIA size Added version number and license to overlay Added chip orientation markers in tdocu layer Repositioned designators
Parts:
- C2: value 10µF -> 10uF
- C21, C22: value NP -> NOT PLACED
- C3, C4: value 47µF -> 47uF
- L1: value 10µH -> 10uH
- R1: value 27 kΩ -> 27K
- R10, R8, R9: value 22Ω -> 22R
- R11, R17, R18: value 10Ω -> 10R
- R12, R19, R20: value 100kΩ -> 100K
- R13, R14: value 0Ω -> 0R
- R15, R16, R2: value 1kΩ -> 1K
- R3: value 12 kΩ -> 12K
- R4, R5, R6, R7: value 10kΩ -> 10K
Other:
- note added: "V1.0 (2013-10-24)"
- note added: "www.freetronics.com/gsmshield"
- note removed: "V0.1 (2013-10-24)"
- note removed: "www.freetronics.com"
